File: Schematics/pi/kicad.kicad_pcb (KiCad board)
At the start: 2 copper layers, 65 x 56 mm, 5 parts, among them P1 Conn_02x20_Odd_Even

Commit message: update2
Parts:
- added U1: keyboard, Seeed-OPL-Connector:H13-2.54, F.Cu at (218.9, 125.2)
- added U2: audio, digikey-footprints:8-DIP, F.Cu at (237.7, 115.6)
Changed lines of the file:
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@@
     (tracks 35)
     (zones 0)
-    (modules 5)
-    (nets 32)
+    (modules 7)
+    (nets 48)
   )
   (page A3)
@@
   (net 30 "/GPIO20(SPI1_MOSI)")
   (net 31 "/GPIO21(SPI1_SCK)")
+  (net 32 "Net-(U1-Pad1)")
+  (net 33 "Net-(U1-Pad2)")
+  (net 34 "Net-(U1-Pad3)")
+  (net 35 "Net-(U1-Pad4)")
+  (net 36 "Net-(U1-Pad5)")
+  (net 37 "Net-(U1-Pad6)")
+  (net 38 "Net-(U1-Pad7)")
+  (net 39 "Net-(U1-Pad8)")
+  (net 40 "Net-(U1-Pad9)")
+  (net 41 "Net-(U1-Pad10)")
+  (net 42 "Net-(U1-Pad11)")
+  (net 43 "Net-(U1-Pad12)")
+  (net 44 "Net-(U2-Pad5)")
+  (net 45 "Net-(U2-Pad6)")
+  (net 46 "Net-(U2-Pad7)")
+  (net 47 "Net-(U2-Pad8)")
   (net_class Default "This is the default net class."
     (clearance 0.2)
@@
     (add_net /ID_SD)
     (add_net GND)
+    (add_net "Net-(U1-Pad1)")
+    (add_net "Net-(U1-Pad10)")
+    (add_net "Net-(U1-Pad11)")
+    (add_net "Net-(U1-Pad12)")
+    (add_net "Net-(U1-Pad2)")
+    (add_net "Net-(U1-Pad3)")
+    (add_net "Net-(U1-Pad4)")
+    (add_net "Net-(U1-Pad5)")
+    (add_net "Net-(U1-Pad6)")
+    (add_net "Net-(U1-Pad7)")
+    (add_net "Net-(U1-Pad8)")
+    (add_net "Net-(U1-Pad9)")
+    (add_net "Net-(U2-Pad5)")
+    (add_net "Net-(U2-Pad6)")
+    (add_net "Net-(U2-Pad7)")
+    (add_net "Net-(U2-Pad8)")
   )
   (net_class Power ""
@@
     (pad 1 np_thru_hole circle (at 0 0 180) (size 2.7 2.7) (drill 2.7) (layers *.Cu *.Mask))
   )
+  (module Seeed-OPL-Connector:H13-2.54 (layer F.Cu)
+    (at 218.893501 125.163501)
+    (fp_text reference U1 (at 0.635 -6.35 90) (layer F.Mask)
+      (effects (font (size 1.2065 1.2065) (thickness 0.127)) (justify left bottom))
+    )
+    (fp_text value keyboard (at 2.54 -2.54 90) (layer F.SilkS)
+      (effects (font (size 0.84455 0.84455) (thickness 0.09779)) (justify left bottom))
+    )
+    (fp_line (start -1.27 -16.51) (end 1.27 -16.51) (layer F.SilkS) (width 0.127))
+    (fp_line (start 1.27 -16.51) (end 1.27 16.51) (layer F.SilkS) (width 0.127))
+    (fp_line (start 1.27 16.51) (end -1.27 16.51) (layer F.SilkS) (width 0.127))
+    (fp_line (start -1.27 16.51) (end -1.27 -16.51) (layer F.SilkS) (width 0.127))
+    (fp_line (start -1.27 -16.51) (end 1.27 -16.51) (layer Dwgs.User) (width 0))
+    (fp_line (start 1.27 -16.51) (end 1.27 16.51) (layer Dwgs.User) (width 0))
+    (fp_line (start 1.27 16.51) (end -1.27 16.51) (layer Dwgs.User) (width 0))
+    (fp_line (start -1.27 16.51) (end -1.27 -16.51) (layer Dwgs.User) (width 0))
+    (fp_poly (pts (xy -1.27 16.51) (xy 1.27 16.51) (xy 1.27 -16.51) (xy -1.27 -16.51)) (layer Dwgs.User) (width 0))
+    (pad 1 thru_hole rect (at 0 -15.24) (size 1.651 1.651) (drill 0.889) (layers *.Cu *.Mask)
+      (net 32 "Net-(U1-Pad1)") (solder_mask_margin 0.1016))
+    (pad 2 thru_hole circle (at 0 -12.7) (size 1.651 1.651) (drill 0.889) (layers *.Cu *.Mask)
+      (net 33 "Net-(U1-Pad2)") (solder_mask_margin 0.1016))
+    (pad 3 thru_hole circle (at 0 -10.16) (size 1.651 1.651) (drill 0.889) (layers *.Cu *.Mask)
+      (net 34 "Net-(U1-Pad3)") (solder_mask_margin 0.1016))
+    (pad 4 thru_hole circle (at 0 -7.62) (size 1.651 1.651) (drill 0.889) (layers *.Cu *.Mask)
+      (net 35 "Net-(U1-Pad4)") (solder_mask_margin 0.1016))
+    (pad 5 thru_hole circle (at 0 -5.08) (size 1.651 1.651) (drill 0.889) (layers *.Cu *.Mask)
+      (net 36 "Net-(U1-Pad5)") (solder_mask_margin 0.1016))
+    (pad 6 thru_hole circle (at 0 -2.54) (size 1.651 1.651) (drill 0.889) (layers *.Cu *.Mask)
+      (net 37 "Net-(U1-Pad6)") (solder_mask_margin 0.1016))
+    (pad 7 thru_hole circle (at 0 0) (size 1.651 1.651) (drill 0.889) (layers *.Cu *.Mask)
+      (net 38 "Net-(U1-Pad7)") (solder_mask_margin 0.1016))
+    (pad 8 thru_hole circle (at 0 2.54) (size 1.651 1.651) (drill 0.889) (layers *.Cu *.Mask)
+      (net 39 "Net-(U1-Pad8)") (solder_mask_margin 0.1016))
+    (pad 9 thru_hole circle (at 0 5.08) (size 1.651 1.651) (drill 0.889) (layers *.Cu *.Mask)
+      (net 40 "Net-(U1-Pad9)") (solder_mask_margin 0.1016))
+    (pad 10 thru_hole circle (at 0 7.62) (size 1.651 1.651) (drill 0.889) (layers *.Cu *.Mask)
+      (net 41 "Net-(U1-Pad10)") (solder_mask_margin 0.1016))
+    (pad 11 thru_hole circle (at 0 10.16) (size 1.651 1.651) (drill 0.889) (layers *.Cu *.Mask)
+      (net 42 "Net-(U1-Pad11)") (solder_mask_margin 0.1016))
+    (pad 12 thru_hole circle (at 0 12.7) (size 1.651 1.651) (drill 0.889) (layers *.Cu *.Mask)
+      (net 43 "Net-(U1-Pad12)") (solder_mask_margin 0.1016))
+    (pad 13 thru_hole circle (at 0 15.24) (size 1.651 1.651) (drill 0.889) (layers *.Cu *.Mask)
+      (net 3 GND) (solder_mask_margin 0.1016))
+  )
+  (module digikey-footprints:8-DIP (layer F.Cu)
+    (at 237.68 115.63)
+    (descr http://media.digikey.com/pdf/Data%20Sheets/Lite-On%20PDFs/6N137%20Series.pdf)
+    (fp_text reference U2 (at 4.05 -2.52) (layer F.SilkS)
+      (effects (font (size 1 1) (thickness 0.15)))
+    )
+    (fp_text value audio (at 3.94 10.33) (layer F.Fab)
+      (effects (font (size 1 1) (thickness 0.15)))
+    )
+    (fp_line (start -1.05 8.89) (end 8.67 8.89) (layer F.CrtYd) (width 0.1))
+    (fp_line (start -1.05 -1.29) (end -1.05 8.89) (layer F.CrtYd) (width 0.1))
+    (fp_line (start 8.67 -1.29) (end 8.67 8.89) (layer F.CrtYd) (width 0.1))
+    (fp_line (start -1.05 -1.29) (end 8.67 -1.29) (layer F.CrtYd) (width 0.1))
+    (fp_line (start 0.4 -0.9) (end 0.4 -1.2) (layer F.SilkS) (width 0.1))
+    (fp_line (start 0.4 -1.2) (end 0.7 -1.2) (layer F.SilkS) (width 0.1))
+    (fp_line (start 7.2 -0.9) (end 7.2 -1.2) (layer F.SilkS) (width 0.1))
+    (fp_line (start 7.2 -1.2) (end 6.9 -1.2) (layer F.SilkS) (width 0.1))
+    (fp_line (start 7.2 8.5) (end 7.2 8.8) (layer F.SilkS) (width 0.1))
+    (fp_line (start 7.2 8.8) (end 6.9 8.8) (layer F.SilkS) (width 0.1))
+    (fp_line (start 0.4 8.5) (end 0.4 8.8) (layer F.SilkS) (width 0.1))
+    (fp_line (start 0.4 8.8) (end 0.7 8.8) (layer F.SilkS) (width 0.1))
+    (fp_line (start 0.55 8.64) (end 7.05 8.64) (layer F.Fab) (width 0.1))
+    (fp_line (start 0.55 -1.04) (end 7.05 -1.04) (layer F.Fab) (width 0.1))
+    (fp_line (start 7.05 -1.04) (end 7.05 8.64) (layer F.Fab) (width 0.1))
+    (fp_line (start 0.55 -1.04) (end 0.55 8.64) (layer F.Fab) (width 0.1))
+    (fp_text user REF** (at 3.94 3.49) (layer F.Fab)
+      (effects (font (size 1 1) (thickness 0.1)))
+    )
+    (pad 1 thru_hole rect (at 0 0) (size 1.6 1.6) (drill 1) (layers *.Cu *.Mask)
+      (net 27 "/GPIO13(PWM1)"))
+    (pad 2 thru_hole circle (at 0 2.54) (size 1.6 1.6) (drill 1) (layers *.Cu *.Mask)
+      (net 2 +5V))
+    (pad 3 thru_hole circle (at 0 5.08) (size 1.6 1.6) (drill 1) (layers *.Cu *.Mask)
+      (net 3 GND))
+    (pad 4 thru_hole circle (at 0 7.62) (size 1.6 1.6) (drill 1) (layers *.Cu *.Mask)
+      (net 20 "/GPIO18(GEN1)(PWM0)"))
+    (pad 5 thru_hole circle (at 7.62 7.62) (size 1.6 1.6) (drill 1) (layers *.Cu *.Mask)
+      (net 44 "Net-(U2-Pad5)"))
+    (pad 6 thru_hole circle (at 7.62 5.08) (size 1.6 1.6) (drill 1) (layers *.Cu *.Mask)
+      (net 45 "Net-(U2-Pad6)"))
+    (pad 7 thru_hole circle (at 7.62 2.54) (size 1.6 1.6) (drill 1) (layers *.Cu *.Mask)
+      (net 46 "Net-(U2-Pad7)"))
+    (pad 8 thru_hole circle (at 7.62 0) (size 1.6 1.6) (drill 1) (layers *.Cu *.Mask)
+      (net 47 "Net-(U2-Pad8)"))
+  )
   (gr_line (start 244 146) (end 244 131) (layer Edge.Cuts) (width 0.1))
